File: KiCad-schematics/iBot Frans.sch (KiCad schematic (older format))
At the start: 3 parts, among them M1 Motor_DC, M2 Motor_DC, U1 arduino_motor_shield

Commit message: modified:   Arduino-scripts/iBot-Frans-drivers/iBot-frans.ino 	modified:   KiCad-schematics/iBot Frans-cache.lib 	modified:   KiCad-schematics/iBot Frans.sch 	modified:   KiCad-schematics/iBot Frans.sch-bak
Parts:
- added SWA, SWB: Rotary_Encoder, symbol Device:Rotary_Encoder
- renumbered M1 to MA, M2 to MB
Connections:
- net at U1.4 (D4): now also SWB.A
- net at U1.5 (D5): now also SWB.B
- net at U1.6 (D6): now also SWA.A
- net at U1.7 (D7): now also SWA.B
Changed lines of the file:
@@
 	4250 2550 4900 2550
 $Comp
-L Motor:Motor_DC M1
+L Motor:Motor_DC MA
 U 1 1 631B4BF5
 P 1900 2550
-F 0 "M1" H 2058 2546 50  0000 L CNN
+F 0 "MA" H 2058 2546 50  0000 L CNN
 F 1 "Motor_DC" H 2058 2455 50  0000 L CNN
 F 2 "" H 1900 2460 50  0001 C CNN
@@
 $EndComp
 $Comp
-L Motor:Motor_DC M2
+L Motor:Motor_DC MB
 U 1 1 631B5CBA
 P 1900 1900
-F 0 "M2" H 2058 1896 50  0000 L CNN
+F 0 "MB" H 2058 1896 50  0000 L CNN
 F 1 "Motor_DC" H 2058 1805 50  0000 L CNN
 F 2 "" H 1900 1810 50  0001 C CNN
@@
 Wire Wire Line
 	1900 2350 4900 2350
+$Comp
+L Device:Rotary_Encoder SWA
+U 1 1 631CF6B4
+P 8550 2250
+F 0 "SWA" H 8780 2296 50  0000 L CNN
+F 1 "Rotary_Encoder" H 8780 2205 50  0000 L CNN
+F 2 "" H 8400 2410 50  0001 C CNN
+F 3 "~" H 8550 2510 50  0001 C CNN
+	1    8550 2250
+	1    0    0    -1
+$EndComp
+$Comp
+L Device:Rotary_Encoder SWB
+U 1 1 631D6520
+P 8550 2800
+F 0 "SWB" H 8780 2846 50  0000 L CNN
+F 1 "Rotary_Encoder" H 8780 2755 50  0000 L CNN
+F 2 "" H 8400 2960 50  0001 C CNN
+F 3 "~" H 8550 3060 50  0001 C CNN
+	1    8550 2800
+	1    0    0    -1
+$EndComp
+Wire Wire Line
+	6050 3550 8050 3550
+Wire Wire Line
+	8150 3450 6050 3450
+Wire Wire Line
+	6050 3350 7850 3350
+Wire Wire Line
+	7950 3250 6050 3250
+Wire Wire Line
+	8150 3450 8150 2900
+Wire Wire Line
+	8150 2900 8250 2900
+Wire Wire Line
+	8050 3550 8050 2700
+Wire Wire Line
+	8050 2700 8250 2700
+Wire Wire Line
+	7950 3250 7950 2350
+Wire Wire Line
+	7850 3350 7850 2150
+Wire Wire Line
+	7950 2350 8250 2350
+Wire Wire Line
+	7850 2150 8250 2150
 $EndSCHEMATC
